Commit message: Fix wrist hand-eye URDF, stop dashboard matching its own API clients
- gen3_macro.xacro: replace the easy_handeye2 camera_module transform (projected the
  gripper pads far outside the wrist image) with the standard Kinova vision-module mount
  (xyz 0 0.05639 0.01305, rpy 0 0 pi); pads now project onto the real fingers.
- process_manager: ignore curl/wget and /api/nodes/ command lines when matching node
  signatures; `curl .../api/nodes/<id>/start` made Start report "already running" and
  `.../stop` killed its own caller.
- RUNBOOK: record the 2026-10-05 camera recalibration and the dry-run route.

Co-Authored-By: Claude Sonnet 5.5 <noreply@anthropic.com>

File: robot_bringup/ros2_kortex/kortex_description/arms/gen3/7dof/urdf/gen3_macro.xacro (robot description, xacro)
@@ -477,6 +477,11 @@
         <link name="${prefix}camera_link" />
         <joint name="${prefix}camera_module" type="fixed">
-          <origin xyz="-0.04943050 0.04958700 0.00395126"
-                  rpy="0.66454839 0.30604363 1.09121110" />
+          <!-- 2026-10-05: the easy_handeye2 result (xyz -0.0494 0.0496 0.0040,
+               rpy 0.6645 0.3061 1.0912) projected the gripper pads far outside the
+               wrist image (real fingers sit in the bottom corners). Replaced by the
+               standard Kinova vision-module mount: 56 mm off the tool axis, optical
+               frame looking along the tool axis (end_effector_link rotated 180 deg about z).
+               That projects the pads to the bottom corners, as in the live image. -->
+          <origin xyz="0 0.05639 0.01305" rpy="0 0 3.14159265358979" />
           <parent link="${prefix}end_effector_link" />
           <child  link="${prefix}camera_link" />
